File: Floe_hw/Floe.kicad_pcb (KiCad board)
At the start: 2 copper layers, 30 x 103 mm, 116 parts, among them Q1 LED_5050, Q2 IRLML6401, Q3 IRLML6401, Q4 IRLML9303, Q5 2N7002, SW1 SWITCH, SW2 BTN, SW3 BTN

Commit message: + simple sch
Parts:
- removed ANT1: ANT_PCB_MONO, Radio:ANT_868_SEIDHE
- removed B1: BAT, Installation:EEMB603030
- removed BLN1: BALUN868JOHANSON, Radio:BALUN_JOHANSON868
- removed C10, C12, C13, C16, C17, C21, C23, C24, C28, C29, C30, C35, C39, C41, C43, C44, C45, C47, C51, C52, C53: 0.1u, Capacitors:CAP_0603
- removed C11, C20, C36, C48: 10u, Capacitors:CAP_0603
- removed C14, C22: 22n, Capacitors:CAP_0603
- removed C15, C18, C19, C25, C26, C27, C31, C32, C33, C34, C40, C7: 1u, Capacitors:CAP_0603
- removed C37, C38: 18pF, Capacitors:CAP_0603
- removed C42, C46: *, Capacitors:CAP_0402
- removed C8, C9: 150pF, Capacitors:CAP_0603
- removed D1: PMEG2020, Diodes:SOD323
- removed DA2: CS42L52, QFN_DFN:QFN40
- removed DA3: NCP583SQ, SOT:SC82AB
- removed DA4: NCP511SN25, SOT:SOT23-5
- removed DD3: LIS3, LGA:LGA16_3X3_5_3
- removed DD4: MMA8452Q, QFN_DFN:QFN16_5x3
- removed F1: Fuse0R, Resistors:RES_0603_FUSE
- removed L1: BLM15, Inductors:IND_0402
- removed L2: BLM15AG102SN1, Inductors:IND_0402
- removed L3: *, Inductors:IND_0402
- removed R18, R19: 100k, Resistors:RES_0603
- removed TP2, TP3, TP4, TP5, TP6, TP7: TESTPOINT, PCB:TESTPOINT_1MM
- removed XL3: CONN_4, Connectors:PLS-4
- removed XL4: AudioJackSimple, Connectors:AUDIO_CKX3_5_30
- removed XL5: CONN_2, Connectors:PLS-2
- removed XL6: CONN_MICROSD, Connectors:MICROSD_CAP_FIX05A
- removed XTAL1: 12MHz, Quartz:0503x4-4
- removed XTAL2: 27MHz, Quartz:03225C4
- added HOLE5: HOLE_METALLED, PCB:Hole3d5_out10mm, F.Cu at (150.0, 36.0)
- added HOLE6: HOLE_METALLED, PCB:Hole3d5_out10mm, F.Cu at (49.4, 57.3)
- added Q6: LED_5050, LEDs:LED_5050, F.Cu at (116.2, 70.6)
- added Q7: LED_5050, LEDs:LED_5050, F.Cu at (184.2, 77.6)
- added SA1: SWITCH_1P2T, BtnsSwitches:SW_SS-1P2T, F.Cu at (73.2, 39.9)
- C1, C3: value 10u -> 0.1u; footprint Capacitors:CAP_0603 -> Capacitors:CAP_0603_Silks
- C2: value 10n -> 10u; footprint Capacitors:CAP_0603 -> Capacitors:CAP_0603_Silks
- C4, C49, C50: footprint Capacitors:CAP_0603 -> Capacitors:CAP_0603_Silks
- C5: value 18pF -> 0.1u; footprint Capacitors:CAP_0603 -> Capacitors:CAP_0603_Silks
- C6: value 18pF -> 10u; footprint Capacitors:CAP_0603 -> Capacitors:CAP_0603_Silks
- DA1: value MCP73832 -> MCP1700; footprint SOT:SOT23-5 -> SOT:SOT23-3A
- DD1: value STM32L476Rx -> STM32F030F6Px; footprint LQFP_TQFP:LQFP64 -> SO_DIL_TSSOP:TSSOP20
- DD2: value CC1101 -> LIS3; footprint QFN_DFN:QFN20 -> LGA:LGA16_3X3_5_3
- HOLE1, HOLE2, HOLE3, HOLE4: footprint PCB:Hole2d4_out4d5mm -> PCB:Hole3d5_out10mm
- Q1: value LED_5050 -> 2N7002; footprint LEDs:LED_5050 -> SOT:SOT23-3; moved to F.Cu
- Q2, Q3: value IRLML6401 -> 2N7002
- Q4: value IRLML9303 -> LED_5050; footprint SOT:SOT23-3 -> LEDs:LED_5050
- Q5: value 2N7002 -> LED_5050; footprint SOT:SOT23-3 -> LEDs:LED_5050
- R1, R2, R3: value 100R -> 10k
- R10, R11: value 51R -> 100R
- R12, R4, R9: value 10k -> 100R
- R13, R14, R5: value 100k -> 100R
- R15: value 20k -> 100R
- R16: value 56k -> 100k
- R6: value 1k -> 100R
- R7, R8: value 4k7 -> 100R
- SW1: value SWITCH -> IT-1187A; footprint BtnsSwitches:SW_SS-1P2T -> BtnsSwitches:BTN_4x4_SMD; moved to F.Cu
- SW2, SW3: value BTN -> IT-1187A; moved to F.Cu
- XL1: footprint Connectors:PLS-6 -> Connectors:PLS-6_LOCK
- XL2: value USB_MINI_B -> CONN_2; footprint Connectors:USBmicro_MOLEX_WM17142 -> Connectors:SLD_2_2D5_1mm
- moved Logo1 138.9 mm to (50.6, 35.5), turned to 0 degrees
- moved XL1 132.6 mm to (46.0, 28.4), turned to 0 degrees
- moved HOLE4 120.9 mm to (60.4, 54.0)
- moved HOLE3 104.2 mm to (154.0, 166.0)
- moved XL7 104.1 mm to (110.0, 28.4)
- moved R16 101.9 mm to (86.2, 45.2)
- moved SW3 98.1 mm to (72.9, 45.5), turned to 0 degrees
- moved R14 95.7 mm to (90.4, 42.6)
- moved HOLE1 91.7 mm to (213.0, 102.0)
- moved SW2 91.0 mm to (82.6, 40.7), turned to 0 degrees
- moved R17 86.4 mm to (78.9, 51.9), turned to 0 degrees
- moved XL2 82.1 mm to (58.0, 61.6), turned to 0 degrees
- moved R6 77.7 mm to (78.9, 54.6), turned to 0 degrees
- moved Q3 76.7 mm to (74.8, 50.6), turned to 0 degrees
- moved C6 76.4 mm to (83.1, 51.9), turned to 0 degrees
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Connections:
- C1 pad 1: GND -> PwrMCU
- C1 pad 2: +5V -> GND
- C2 pad 2: +5V -> PwrMCU
- C3 pad 1: GND -> PwrMCU
- C3 pad 2: +BATT -> GND
- C4 pad 1: VAA -> +BATT
- C49 pad 1: PwrMCU -> /ACC_PWR
- C5 pad 1: Net-(C5-Pad1) -> PwrMCU
- C50 pad 1: VCC -> /ACC_PWR
- C6 pad 1: Net-(C6-Pad1) -> GND
- C6 pad 2: GND -> +BATT
- DA1 pad 1: /Charge -> GND
- DA1 pad 2: GND -> PwrMCU
- DD1 pad 1: PwrMCU -> GND
- DD1 pad 10: (no net) -> /LEDR_CTRL
- DD1 pad 11: /AU_SDIN -> /ACC_PWR
- DD1 pad 12: GND -> /LEDG_CTRL
- DD1 pad 13: PwrMCU -> /LEDB_CTRL
- DD1 pad 14: /BTN_UP -> /BTN1
- DD1 pad 15: /BTN_DOWN -> GND
- DD1 pad 16: (no net) -> PwrMCU
- DD1 pad 17: /CC_GDO0 -> /I2C_SCL
- DD1 pad 18: GND -> /I2C_SDA
- DD1 pad 19: PwrMCU -> /SWDIO
- DD1 pad 2: (no net) -> /ACC_INT1
- DD1 pad 20: /CC_CS -> /SWCLK
- DD1 pad 3: (no net) -> /BTN2
- DD1 pad 5: Net-(C5-Pad1) -> PwrMCU
- DD1 pad 6: Net-(DD1-Pad6) -> /BTN0
- DD1 pad 7: (no net) -> /BAT_MEAS
- DD1 pad 8: (no net) -> /UART_TX
- DD1 pad 9: (no net) -> /UART_RX
- DD2 pad 1: /CC_SCK -> /ACC_PWR
- DD2 pad 10: Net-(C38-Pad1) -> GND
- DD2 pad 11: VCC -> /ACC_INT1
- DD2 pad 12: /RF1 -> GND
- DD2 pad 13: /RF2 -> (no net)
- DD2 pad 14: VCC -> /ACC_PWR
- DD2 pad 15: VCC -> (no net)
- DD2 pad 16: GND -> (no net)
- DD2 pad 2: /CC_MISO -> (no net)
- DD2 pad 4: VCC -> /I2C_SCL
- DD2 pad 5: Net-(C39-Pad2) -> GND
- DD2 pad 6: /CC_GDO0 -> /I2C_SDA
- DD2 pad 7: /CC_CS -> /ACC_PWR
- DD2 pad 8: Net-(C37-Pad1) -> /ACC_PWR
- DD2 pad 9: VCC -> (no net)
- Q1 pad 1: Net-(Q1-Pad1) -> /LEDR_CTRL
- Q1 pad 2: Net-(Q1-Pad2) -> GND
- Q1 pad 3: Net-(Q1-Pad3) -> /LED_R
- Q2 pad 1: +5V -> /LEDG_CTRL
- Q2 pad 2: /PWR_UNST_ALWAYS -> GND
- Q2 pad 3: +BATT -> /LED_G
- Q3 pad 1: /PWR_EN -> /LEDB_CTRL
- Q3 pad 2: PwrUnst -> GND
- Q3 pad 3: /PWR_CTRLED -> /LED_B
- Q4 pad 1: /SD_PWR_EN -> +BATT
- Q4 pad 2: +3.3V -> +BATT
- Q4 pad 3: /SD_PWR -> +BATT
- Q5 pad 1: /MEASURE_EN -> +BATT
- Q5 pad 2: GND -> +BATT
- Q5 pad 3: Net-(Q5-Pad3) -> +BATT
- R1 pad 1: Net-(Q1-Pad1) -> /BTN0
- R1 pad 2: /BLUE_LED -> GND
- R10 pad 1: GND -> /LED_B
- R11 pad 1: GND -> /LED_B
- R12 pad 1: Net-(DD1-Pad41) -> /LED_R
- R12 pad 2: +5V -> Net-(Q6-Pad5)
- R13 pad 1: /PWR_EN -> /LED_R
- R13 pad 2: PwrUnst -> Net-(Q7-Pad5)
- R14 pad 1: +3.3V -> /LED_G
- R14 pad 2: /SD_PWR_EN -> Net-(Q6-Pad4)
- R15 pad 1: /CC_CS -> /LED_G
- R15 pad 2: VCC -> Net-(Q7-Pad4)
- R16 pad 1: Net-(DD2-Pad17) -> /BAT_MEAS
- R16 pad 2: GND -> +BATT
- R17 pad 2: /MEASURE_EN -> /BAT_MEAS
- R2 pad 1: Net-(Q1-Pad2) -> /ACC_PWR
- R2 pad 2: /RED_LED -> /I2C_SCL
- R3 pad 1: Net-(Q1-Pad3) -> /I2C_SDA
- R3 pad 2: /GREEN_LED -> /ACC_PWR
- R4 pad 1: Net-(DA1-Pad5) -> /LED_B
- R4 pad 2: GND -> Net-(Q4-Pad6)
- R5 pad 1: GND -> /LED_B
- R5 pad 2: /AU_RST -> Net-(Q5-Pad6)
- R6 pad 1: Net-(C6-Pad1) -> /LED_R
- R6 pad 2: Net-(DD1-Pad6) -> Net-(Q4-Pad5)
- R7 pad 1: /SDA -> /LED_R
- R7 pad 2: VAA -> Net-(Q5-Pad5)
- R8 pad 1: /SCL -> /LED_G
- R8 pad 2: VAA -> Net-(Q4-Pad4)
- R9 pad 1: +5V -> /LED_G
- R9 pad 2: GND -> Net-(Q5-Pad4)
- SW1 pad 1: PwrUnst -> PwrMCU
- SW1 pad 2: /PWR_UNST_ALWAYS -> /BTN0
- SW2 pad 1: /BTN_UP -> PwrMCU
- SW2 pad 2: PwrMCU -> /BTN1
- SW3 pad 1: /BTN_DOWN -> PwrMCU
- SW3 pad 2: PwrMCU -> /BTN2
- XL2 pad 1: +5V -> GND
- XL2 pad 2: /D- -> Net-(SA1-Pad2)
Routing:
- net GND: track 648.1 -> 19.4 mm, vias 116 -> 0
- net /ANT2: track 142.0 -> 0.00 mm
- net PwrMCU: track 158.5 -> 22.0 mm, vias 13 -> 2
- net VCC: track 59.9 -> 0.00 mm, vias 6 -> 0
- net VAA: track 58.3 -> 0.00 mm, vias 5 -> 0
- net /SDA: track 51.0 -> 0.00 mm, vias 4 -> 0
- net /D-: track 48.4 -> 0.00 mm, vias 2 -> 0
- net /D+: track 47.4 -> 0.00 mm, vias 2 -> 0
- net /SCL: track 47.2 -> 0.00 mm, vias 4 -> 0
- net /RED_LED: track 44.7 -> 0.00 mm, vias 2 -> 0
- net /GREEN_LED: track 42.7 -> 0.00 mm, vias 2 -> 0
- net +5V: track 40.4 -> 0.00 mm, vias 2 -> 0
- net PwrUnst: track 38.1 -> 0.00 mm, vias 1 -> 0
- net /PWR_CTRLED: track 32.7 -> 0.00 mm, vias 2 -> 0
- net /BLUE_LED: track 32.3 -> 0.00 mm, vias 2 -> 0
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- removed copper zone on B.Cu, net GND
- removed copper zone on F.Cu, net GND
Other:
- board size 30 x 103 mm -> 140 x 140 mm
- board text removed: "+"
- board text removed: "-"
- board text removed: "Bat measure"
- board text removed: "Charger"
- board text removed: "GND"
- board text removed: "LRCK"
- board text removed: "MCLK"
- board text removed: "Off On"
- board text removed: "Ostranna Quendelasse"
- board text removed: "PB13"
- board text removed: "PB14"
- board text removed: "PB15"
- board text removed: "SCLK"
- board text removed: "SDIN"
- board text removed: "SDOUT"
- board text removed: "Speaker"
