File: Floe_hw/Floe.kicad_sch (KiCad schematic)
At the start: 154 parts, among them Q1 IRLML6401, Q2 IRF9317, Q3 LED_5050, Q4 2N7002, Q5 IRLML6401, Q6 IRLML6401, Q7 IRLML6401, Q8 2N7002

Commit message: + simple sch
Parts:
- removed ANT1: ANT_GENERAL, Antennas:ANT_868_IFA_SIMPLEJOY, symbol Antennas_kl:ANT_GENERAL
- removed B1: BAT, Installation:EEMB603030, symbol Power_kl:BAT
- removed C10, C11, C12, C35, C36, C37, C39, C42, C44, C45, C53, C54, C55, C57, C58, C59, C9: 0.1u, Capacitors:CAP_0603, symbol Tittar_kl:C
- removed C13, C20, C22, C34, C38, C56, C60, C63, C64, C65: 1u, Capacitors:CAP_0603, symbol Tittar_kl:C
- removed C14, C15, C26, C43, C52, C61, C62, C66: 10u, Capacitors:CAP_0603, symbol Tittar_kl:C
- removed C16: 47pFpF, Capacitors:CAP_0402, symbol Tittar_kl:C
- removed C17, C30: 47pF, Capacitors:CAP_0402, symbol Tittar_kl:C
- removed C18, C19: C, Capacitors:CAP_0402, symbol Tittar_kl:C
- removed C21, C8: 3.3pF, Capacitors:CAP_0402, symbol Tittar_kl:C
- removed C23, C24: 1000pF, Capacitors:CAP_0402, symbol Tittar_kl:C
- removed C25, C33: 150pF, Capacitors:CAP_0603, symbol Tittar_kl:C
- removed C27, C28, C29, C31, C32: 0.1u, Capacitors:CAP_0402, symbol Tittar_kl:C
- removed C40, C41: 18pF, Capacitors:CAP_0603_Silks, symbol Tittar_kl:C
- removed C46, C47: 18pF, Capacitors:CAP_0603, symbol Tittar_kl:C
- removed C48: 0.1u, Capacitors:CAP_0603_Silks, symbol Tittar_kl:C
- removed C51: 10n, Capacitors:CAP_0603, symbol Tittar_kl:C
- removed C7: 8.2pF, Capacitors:CAP_0402, symbol Tittar_kl:C
- removed D1: PMEG2020, Diodes:SOD323, symbol Tittar_kl:D_Shottky
- removed DA1: CS42L52, QFN_DFN:QFN40, symbol Audio_kl:CS42L52
- removed DA2: PE4259, SOT:SC70, symbol RF_ICs:PE4259
- removed DA3: MC74VHC1, SOT:SOT23-5, symbol standard_logic:1xBUF_W3STATE
- removed DA4: TP4056, SO_DIL_TSSOP:SO8_150MIL, symbol Power_kl:TP4056
- removed DA5: MCP1700, SOT:SOT23-3A, symbol Power_kl:MCP1700
- removed DA6: NCP511SN25, SOT:SOT23-5, symbol Power_kl:TPS763xx
- removed DD1: SX1276, QFN_DFN:QFN-28_EP_6x6_Pitch0.65mm, symbol RF_ICs:SX1276
- removed DD2: W25Q128, SO_DIL_TSSOP:SO8_208MIL, symbol memory:W25Q32JV
- removed DD3: MMA8452Q, QFN_DFN:QFN16_5x3, symbol Sensors:MMA8452Q
- removed DD4: STM32L476Rx, LQFP_TQFP:LQFP64, symbol st_kl:STM32L476Rx
- removed DD5: LIS3, symbol Sensors:LIS3
- removed L1: 33nH, Inductors:IND_0402, symbol Tittar_kl:L
- removed L2: 2.2nH, Inductors:IND_0402, symbol Tittar_kl:L
- removed L3: 5.6nH, Inductors:IND_0402, symbol Tittar_kl:L
- removed L4: 4.7nH, Inductors:IND_0402, symbol Tittar_kl:L
- removed L5: L, Inductors:IND_0402, symbol Tittar_kl:L
- removed L6: 10nH, Inductors:IND_0402, symbol Tittar_kl:L
- removed L7: Choke, Inductors:IND_0402, symbol Tittar_kl:L
- removed L8: BLM15, Inductors:IND_0402, symbol Tittar_kl:L
- removed MIC1, MIC2: MSM261D3526Z1CM, Microphones:SPH0644, symbol Audio_kl:PDM_MIC_SPH0644
- removed Q1, Q5, Q6, Q7: IRLML6401, SOT:SOT23-3, symbol Transistors_kl:P_3PIN
- removed Q2: IRF9317, SO_DIL_TSSOP:SO8_150MIL, symbol Transistors_kl:P_8PIN
- removed Q3: LED_5050, LEDs:LED_5050, symbol Tittar_kl:LED_5050
- removed Q4, Q8: 2N7002, SOT:SOT23-3, symbol Transistors_kl:N_3PIN
- removed R18, R20, R24: 100k, Resistors:RES_0603, symbol Tittar_kl:R
- removed R19: 0R2, Resistors:RES_1206, symbol Tittar_kl:R
- removed R21, R23: 10k, Resistors:RES_0603, symbol Tittar_kl:R
- removed R22: 1.2k, Resistors:RES_0603, symbol Tittar_kl:R
- removed SA1: SS9, BtnsSwitches:SW_SS9, symbol BtnsSwitches:SWITCH_1P2T_housing
- removed TP1, TP10, TP11, TP12, TP13, TP14, TP15, TP16, TP17, TP2, TP3, TP4, TP5, TP6, TP7, TP8, TP9: TESTPOINT, PCB:TESTPOINT_1MM, symbol pcb_details:TESTPOINT
- removed XL1: CONN_2, Connectors:WB-02(MW-2M), symbol Connectors_kl:CONN_2
- removed XL3: CONN_4, Connectors:PLS-4, symbol Connectors_kl:CONN_4
- removed XL4: CONN_6, Connectors:PLS-6, symbol Connectors_kl:CONN_6
- removed XL5: USB_MINI_B, Connectors:USBmicro_MOLEX_WM17142, symbol Connectors_kl:USB_MINI_B
- removed XL6: CONN_3, Connectors:SLD_3_2D5, symbol Connectors_kl:CONN_3
- removed XTAL1: 32MHz, Quartz:03225C4, symbol Tittar_kl:CRYSTAL_H
- removed XTAL2: 12MHz, Quartz:0503x4-4, symbol Tittar_kl:CRYSTAL_H
- added DA1: MCP1700, SOT:SOT23-3A, symbol Power_kl:MCP1700
- added DD1: STM32F030F6Px, SO_DIL_TSSOP:TSSOP20, symbol st_kl:STM32F030F6Px
- added DD2: LIS3, LGA:LGA16_3X3_5_3, symbol Sensors:LIS3
- added HOLE5, HOLE6: HOLE_METALLED, PCB:Hole3d5_out10mm, symbol pcb_details:HOLE_METALLED
- added Q1, Q2, Q3: 2N7002, SOT:SOT23-3, symbol Transistors_kl:N_3PIN
- added Q4, Q5, Q6, Q7: LED_5050, LEDs:LED_5050, symbol Tittar_kl:LED_5050
- added SA1: SWITCH_1P2T, BtnsSwitches:SW_SS-1P2T, symbol BtnsSwitches:SWITCH_1P2T
- added SW1, SW2, SW3: IT-1187A, BtnsSwitches:BTN_4x4_SMD, symbol BtnsSwitches:BUTTON
- added XL1: CONN_6, Connectors:PLS-6_LOCK, symbol Connectors_kl:CONN_6
- C1: value 10n -> 0.1u; footprint Capacitors:CAP_0402 -> Capacitors:CAP_0603_Silks
- C2: value 47pF -> 10u; footprint Capacitors:CAP_0402 -> Capacitors:CAP_0603_Silks; PN (none) -> CL10A106MQ8NNNC; Price (none) -> 2.5; SolderPoints (none) -> 2; URL (none) -> https://www.terraelectronica.ru/catalog.php?ID=1155&search=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
- C3: value 1.5pF -> 0.1u; footprint Capacitors:CAP_0402 -> Capacitors:CAP_0603_Silks
- C4: value 22pF -> 0.1u; footprint Capacitors:CAP_0402 -> Capacitors:CAP_0603_Silks; Price (none) -> 0.5; SolderPoints (none) -> 2
- C49, C50: footprint Capacitors:CAP_0603 -> Capacitors:CAP_0603_Silks
- C5: value 1u -> 0.1u; footprint Capacitors:CAP_0603 -> Capacitors:CAP_0603_Silks
- C6: value 8.2pF -> 10u; footprint Capacitors:CAP_0402 -> Capacitors:CAP_0603_Silks; PN (none) -> CL10A106MQ8NNNC; Price (none) -> 2.5; SolderPoints (none) -> 2; URL (none) -> https://www.terraelectronica.ru/catalog.php?ID=1155&search=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
- HOLE1, HOLE2, HOLE3, HOLE4: footprint PCB:Hole2d4_out4d5mm -> PCB:Hole3d5_out10mm
- R1: value 100k -> 10k; Price (none) -> 0.5; SolderPoints (none) -> 2
- R10: value 10k -> 100R; PN (none) -> -; Tolerance (none) -> 1%; Type (none) -> Resistor
- R11, R12, R13, R15, R4: value 1k -> 100R; PN (none) -> -; Tolerance (none) -> 1%; Type (none) -> Resistor
- R14: value 10k -> 100R; PN (none) -> -; Price (none) -> 0.5; SolderPoints (none) -> 2; Tolerance (none) -> 1%; Type (none) -> Resistor
- R16, R17: Price (none) -> 0.5; SolderPoints (none) -> 2
- R2, R3: value 33R -> 10k; footprint Resistors:RES_0402_sm -> Resistors:RES_0603; Price 0.5 -> (none); SolderPoints 2 -> (none)
- R5, R6: value 33R -> 100R; footprint Resistors:RES_0402_sm -> Resistors:RES_0603; PN (none) -> -; Tolerance (none) -> 1%; Type (none) -> Resistor
- R7, R8: value 4k7 -> 100R; PN (none) -> -; Tolerance (none) -> 1%; Type (none) -> Resistor
- R9: value 100k -> 100R; PN (none) -> -; Price (none) -> 0.5; SolderPoints (none) -> 2; Tolerance (none) -> 1%; Type (none) -> Resistor
- XL2: footprint Connectors:W02_Pitch_2d54 -> Connectors:SLD_2_2D5_1mm
Connections:
- net +3v3 is gone; now on net LED_G: R9.1
- net AU_RST is gone; now on net GND: R1.2
- net NPX_PWR_EN is gone; now on net +BATT: R16.2
- net PDM_IN6 is gone; now on net LED_R: R6.1
- net SCL is gone; now on net LED_G: R8.1
- net SDA is gone; now on net LED_R: R7.1
- net +BATT: now also C4.1, C6.2, DA1.3 (IN), Q4.1, Q4.2, Q4.3, Q5.1, Q5.2, Q5.3, Q6.1, Q6.2, Q6.3, Q7.1, Q7.2, Q7.3, SA1.1; no longer R14.1, R17.1
- net ACC_INT1: now also DD1.2 (PF0/OSCIN), DD2.11 (INT1)
- net BAT_MEAS: now also R16.1, DD1.7 (ADC1/PA1)
- net GND: now also C2.1, C3.2, C4.2, C5.2, C6.1, R17.1, DA1.1 (GND), DD1.1 (BOOT0), DD1.15 (VSS), DD2.10 (Reserved), DD2.12 (GND), DD2.5 (GND), HOLE5.H, HOLE6.H, Q1.2 (S), Q2.2 (S), Q3.2 (S), XL1.3; no longer C2.2, C6.2, R1.1, R16.1
- net PwrMCU: now also C1.1, C2.2, C3.1, C5.1, DA1.2 (OUT), DD1.16 (VDD), DD1.5 (VDDA), SW1.1, SW2.1, SW3.1, XL1.1; no longer C49.1, C50.1
- net SWCLK: now also DD1.20 (SWCLK/PA14), XL1.2
- net SWDIO: now also DD1.19 (IR_OUT/SWDIO/PA13), XL1.4
- net UART_RX: now also DD1.9 (ADC3/RX1/PA3), XL1.6
- net UART_TX: now also DD1.8 (ADC2/TX1/PA2), XL1.5
- net at R12.2: now also Q6.5 (G)
- net at R13.2: now also Q7.5 (G)
- net at R15.2: now also Q7.4 (B)
- net LED_B: now reaches R10.1
- net LED_B: now also R11.1, R4.1, R5.1, Q3.3 (D)
- net at R11.2: now also Q7.6
- net LED_R: now reaches R12.1
- net LED_R: now also R13.1, Q1.3 (D)
- net LED_G: now reaches R15.1
- net LED_G: now also R14.1, Q2.3 (D)
- net at R14.2: now also Q6.4 (B)
- net ACC_PWR: now reaches R3.2
- net ACC_PWR: now also C49.1, C50.1, R2.1, DD1.11 (ADC5/SCK1/PA5), DD2.1 (VddIO), DD2.14 (Vdd), DD2.7 (SDO(SA0)), DD2.8 (CS)
- net at R6.2: now also Q4.5 (G)
- net at R5.2: now also Q5.6
- net at R4.2: now also Q4.6
- net I2C_SCL: now reaches R2.2
- net I2C_SCL: now also DD1.17 (TX1/SCL1/T1C2/PA9), DD2.4 (SCL(SPC))
- net +5v: no longer names the net of R10.2
- net +5v: now also Q6.6
- net Btn0: no longer names the net of XL2.2 (PM)
- net Btn0: now also SA1.2
- net MEM_PWR_EN: no longer names the net of R9.2
- net MEM_PWR_EN: now also Q5.4 (B)
- removed net PDM_CLK: R2.1, R5.1
- net PDM_IN2 renamed I2C_SDA
- net I2C_SDA: now also DD1.18 (RX1/SDA1/T1C3/PA10), DD2.6 (SDA(SDI/SDO))
- net VAA: no longer names the net of R7.2
- net VAA: now also Q5.5 (G); no longer R8.2
- new net: Q4.4 (B), R8.2
- new net BTN0: DD1.6 (ADC0/WKUP1/PA0), R1.1, SW1.2
- new net BTN1: DD1.14 (PB1/T3C4/T14C1/T1C3N/ADC9), SW2.2
- new net BTN2: DD1.3 (PF1/OSCOUT), SW3.2
- new net LEDB_CTRL: DD1.13 (ADC7/MOSI1/T3C2/T14C1/T1C1N/T17C1/PA7), Q3.1 (G)
- new net LEDG_CTRL: DD1.12 (ADC6/MISO1/T3C1/T16C1/PA6), Q2.1 (G)
- new net LEDR_CTRL: DD1.10 (ADC4/T14C1/PA4), Q1.1 (G)
- no-connect marks 31 -> 6
Other:
- note added: "Accelerometer"
- note added: "Periphery T2 C1,2,3,4: LEDs I2C1: MEMS Sns UART1: Debug UART DMA C1: ADC C2: USART1 TX C3: USART1 RX C6: I2C1 TX C7: I2C1 RX"
- note removed: "1.6 to 5V"
- note removed: "1.8 to 2.5V"
- note removed: "1.8 to 3.3V"
- note removed: "Accelerometers"
- note removed: "Audio"
- note removed: "Battery or USB"
- note removed: "Buffer"
- note removed: "Button"
- note removed: "Charger 1.2k => 1000mA"
- note removed: "Flash"
- note removed: "I2C addr = 0x1C"
- note removed: "Just pins"
- note removed: "LORA radio"
- note removed: "MCO"
- note removed: "MCU Power Filter"
- note removed: "MCU power"
- note removed: "Maybe this one is acceptable: 50 mOhm"
- note removed: "Mics"
- note removed: "Neopixel"
- note removed: "One or another"
- note removed: "Pins 19 32 48 64 1 13"
- note removed: "RGB LED"
- note removed: "USB Detect"
- note removed: "WKUP2"
- moved on the sheet: C49, C50, HOLE1, HOLE2, HOLE3, Logo1, XL7
