File: Floe_hw/Floe.kicad_sch (KiCad schematic)
At the start: 115 parts, among them Q1 LED_5050, Q2 IRLML6401, Q3 IRLML6401, Q5 2N7002, SW1 SWITCH

Commit message: + Sch seems done
Parts:
- removed ANT?: ANT_PCB_MONO_2PIN, symbol Antennas_kl:ANT_PCB_MONO_2PIN
- removed BLN?: BALUN868JOHANSON, Radio:BALUN_JOHANSON868, symbol RF_ICs:BALUN868JOHANSON
- removed C22: 22n, Capacitors:CAP_0603, symbol Tittar_kl:C
- removed C35, C43, C44, C45, C47, C50: 0.1u, Capacitors:CAP_0603, symbol Tittar_kl:C
- removed C37, C38: 18pF, Capacitors:CAP_0603, symbol Tittar_kl:C
- removed C46: *, Capacitors:CAP_0402, symbol Tittar_kl:C
- removed DD?: CC1101, QFN_DFN:QFN20, symbol RF_ICs:CC1101
- removed R10, R11: 51R, Resistors:RES_0603, symbol Tittar_kl:R
- removed R15: 56k, Resistors:RES_0603, symbol Tittar_kl:R
- removed SW1: SWITCH, BtnsSwitches:SW_SS-1P2T, symbol Switches:SWITCH_1P2T
- removed TP?: TESTPOINT, PCB:TESTPOINT_1MM, symbol pcb_details:TESTPOINT
- removed XL4: AudioJackSimple, Connectors:AUDIO_CKX3_5_30, symbol Connectors_kl:AudioJackSimple
- removed XTAL2: 27MHz, Quartz:03225C4, symbol Tittar_kl:CRYSTAL_H
- added ANT1: ANT_GENERAL, Antennas:ANT_868_IFA_SIMPLEJOY, symbol Antennas_kl:ANT_GENERAL
- added C1: 10n, Capacitors:CAP_0402, symbol Tittar_kl:C
- added C15: 10u, Capacitors:CAP_0603, symbol Tittar_kl:C
- added C16: 47pFpF, Capacitors:CAP_0402, symbol Tittar_kl:C
- added C17, C2, C30: 47pF, Capacitors:CAP_0402, symbol Tittar_kl:C
- added C18, C19: C, Capacitors:CAP_0402, symbol Tittar_kl:C
- added C21, C8: 3.3pF, Capacitors:CAP_0402, symbol Tittar_kl:C
- added C23, C24: 1000pF, Capacitors:CAP_0402, symbol Tittar_kl:C
- added C27, C28, C29, C31, C32: 0.1u, Capacitors:CAP_0402, symbol Tittar_kl:C
- added C3: 1.5pF, Capacitors:CAP_0402, symbol Tittar_kl:C
- added C4: 22pF, Capacitors:CAP_0402, symbol Tittar_kl:C
- added C48: 0.1u, Capacitors:CAP_0603_Silks, symbol Tittar_kl:C
- added C6, C7: 8.2pF, Capacitors:CAP_0402, symbol Tittar_kl:C
- added C9: 0.1u, Capacitors:CAP_0603, symbol Tittar_kl:C
- added DA2: PE4259, SOT:SC70, symbol RF_ICs:PE4259
- added DA3: MC74VHC1, SOT:SOT23-5, symbol standard_logic:1xBUF_W3STATE
- added DD1: SX1276, QFN_DFN:QFN-28_EP_6x6_Pitch0.65mm, symbol RF_ICs:SX1276
- added DD2: W25Q128, SO_DIL_TSSOP:SO8_208MIL, symbol memory:W25Q32JV
- added L1: 33nH, Inductors:IND_0402, symbol Tittar_kl:L
- added L4: 4.7nH, Inductors:IND_0402, symbol Tittar_kl:L
- added L5: L, Inductors:IND_0402, symbol Tittar_kl:L
- added L6: 10nH, Inductors:IND_0402, symbol Tittar_kl:L
- added L7: Choke, Inductors:IND_0402, symbol Tittar_kl:L
- added MIC1, MIC2: MSM261D3526Z1CM, Microphones:SPH0644, symbol Audio_kl:PDM_MIC_SPH0644
- added Q2: IRF9317, SO_DIL_TSSOP:SO8_150MIL, symbol Transistors_kl:P_8PIN
- added Q4: 2N7002, SOT:SOT23-3, symbol Transistors_kl:N_3PIN
- added Q5: IRLML6401, SOT:SOT23-3, symbol Transistors_kl:P_3PIN
- added R14: 10k, Resistors:RES_0603, symbol Tittar_kl:R
- added R2, R3, R5, R6: 33R, Resistors:RES_0402_sm, symbol Tittar_kl:R
- added R4: 1k, Resistors:RES_0603, symbol Tittar_kl:R
- added SA1: SS9, BtnsSwitches:SW_SS9, symbol BtnsSwitches:SWITCH_1P2T_housing
- added TP1, TP10, TP12, TP14, TP17, TP2, TP3, TP5, TP6, TP8, TP9: TESTPOINT, PCB:TESTPOINT_1MM, symbol pcb_details:TESTPOINT
- added XL2: CONN_2, Connectors:W02_Pitch_2d54, symbol Connectors_kl:CONN_2
- added XL6: CONN_3, Connectors:SLD_3_2D5, symbol Connectors_kl:CONN_3
- added XTAL1: 32MHz, Quartz:03225C4, symbol Tittar_kl:CRYSTAL_H
- C14: value 22n -> 10u; Price 0.5 -> (none); SolderPoints 2 -> (none)
- C40: value 1u -> 18pF; footprint Capacitors:CAP_0603 -> Capacitors:CAP_0603_Silks; Price (none) -> 0.5; SolderPoints (none) -> 2
- C41: value 0.1u -> 18pF; footprint Capacitors:CAP_0603 -> Capacitors:CAP_0603_Silks; Price (none) -> 0.5; SolderPoints (none) -> 2
- C42: value * -> 0.1u; footprint Capacitors:CAP_0402 -> Capacitors:CAP_0603; Price 0.5 -> (none); SolderPoints 2 -> (none)
- L2: value BLM15AG102SN1 -> 2.2nH; Price (none) -> 4; SolderPoints (none) -> 2
- L3: value * -> 5.6nH
- R12: renamed from R1; value 100R -> 1k
- R13: renamed from R2; value 100R -> 1k
- R15: renamed from R3; value 100R -> 1k
- R16: value 56k -> 100k; Price 0.5 -> (none); SolderPoints 2 -> (none)
- gave numbers to parts that had none: 13
- renumbered C4 to C10, C16 to C11, C23 to C12, C26 to C13, C18 to C20, C19 to C22, C8 to C25, C20 to C26, C9 to C33, C7 to C34, C10 to C35, C17 to C36, C24 to C37, C27 to C38, C49 to C43, C52 to C44, C53 to C45, C5 to C46, C6 to C47, C48 to C49, C15 to C5, C51 to C50, C2 to C51, C11 to C52, C12 to C53, C13 to C54, C21 to C55, C25 to C56, C28 to C57, C29 to C58, C30 to C59, C31 to C60, C34 to C65, C36 to C66, DA4 to DA6, DD1 to DD4, L1 to L8, Q1 to Q3, Q3 to Q6, Q2 to Q7, Q5 to Q8, R5 to R1, R12 to R10, R6 to R11, R18 to R17, R13 to R18, R19 to R20, R9 to R23, R17 to R24, R14 to R9, TP2 to TP11, TP3 to TP13, TP5 to TP15, TP6 to TP16, XL5 to XL1, XL1 to XL4, XL2 to XL5, XTAL1 to XTAL2
Connections:
- net AU_SDOUT is gone; now on net SX_DIO2: TP4.1
- net BLUE_LED is gone; now on an unnamed net: R12.2
- net CC_GDO0 is gone; now on net SX_MISO: TP7.1
- net GREEN_LED is gone; now on an unnamed net: R15.2
- net PWR_CTRLED is gone; now on net AU_PWR: C11.1, C12.1, C13.1, C65.1, DA1.5 (VP), DA1.8 (VP), DA6.1 (IN), DA6.3 (EN), Q6.3 (D)
- net RED_LED is gone; now on an unnamed net: R13.2
- net +3v3: now also L7.2; no longer L2.2
- net +BATT: now also Q2.1 (S), Q2.2 (S), Q2.3 (S), Q5.2 (S), R14.1
- net AU_RST: now also DD4.11 (ADC123-4/MOSI2/PC3); no longer DD4.35 (PB14/MISO2/SDA2/T15C1)
- net BAT_MEAS: now also DD4.20 (ADC12-9/LPTIM2_OUT/DAC1/CK2/PA4)
- net ChrgEn: now also DD4.4 (OC32OUT/PC15)
- net GND: now also C14.2, R16.1, ANT1.2 (GND), C1.2, C15.2, C18.2, C19.2, C2.2, C21.2, C23.2, C24.2, C27.2, C28.2, C29.2, C30.2, C31.2, C32.2, C48.1, C6.2, C7.2, C8.2, C9.1, DA2.2 (GND), DA3.1 (~OE), DA3.3 (GND), DD1.15 (GND), DD1.23 (GND), DD1.26 (GND), DD1.PAD (GND), DD2.4 (GND), MIC1.2 (SELECT), MIC1.3 (GND), MIC2.2 (SELECT), MIC2.3 (GND), Q4.2 (S), SA1.H, XL2.1 (P1), XL6.1 (P1), XTAL1.H; no longer R16.2
- net IsCharging: now also DD4.3 (OC32IN/PC14)
- net MEASURE_EN: now also DD4.21 (ADC12-10/T2C1/DAC2/SCK1/PA5)
- net PWR_UNST_ALWAYS: now also SA1.2
- net PwrUnst: now also SA1.1
- net QSPI_CLK: now also DD2.6 (CLK)
- net QSPI_IO0: now also DD2.5 (DI/IO0)
- net QSPI_IO1: now also DD2.2 (DO/IO1)
- net QSPI_IO2: now also DD2.3 (IO2)
- net QSPI_IO3: now also DD2.7 (IO3)
- net QSPI_NCS: now also DD2.1 (~CS)
- net VCC: now also C24.1, C27.1, C28.1, C29.1, C30.1, DA2.6 (VDD), DD1.14 (VBAT_DIG), DD1.24 (VBAT_RF), DD1.3 (VBAT_ANA), L7.1; no longer C40.1, C41.1, L2.1
- net AU_PWR: now reaches C14.1
- net AU_PWR: now also C15.1
- net PDM_CLK: now reaches DD4.10 (ADC123-3/LPTIM1_IN2/MISO2/PC2)
- net PDM_CLK: now also R2.1, R5.1, TP10.1
- net SX_DIO1: now reaches DD4.15 (ADC12-6/T2C2/T5C2/RX4/PA1)
- net SX_DIO1: now also DD1.9 (DIO1/DCLK), TP3.1
- net SX_DIO2: now reaches DD4.16 (ADC12-7/WKUP4/T15C1/T2C3/T5C3/TX2/PA2)
- net SX_DIO2: now also DD1.10 (DIO2/DATA)
- net SX_DIO3: now reaches DD4.17 (ADC12-8/T15C2/T2C4/T5C4/RX2/PA3)
- net SX_DIO3: now also DD1.11 (DIO3), TP5.1
- net at DD4.24 (ADC12-13/TX3/PC4): now also XL3.3
- net at DD4.25 (ADC12-14/RX3/PC5): now also XL3.4
- net MEM_PWR_EN: now reaches DD4.28 (PB2/LPTIM1_OUT/RTC_OUT)
- net MEM_PWR_EN: now also Q1.1 (G), R9.2
- net MIC_VDD: now reaches DD4.40 (OTG_NOE/T3C4/T8C4/SDIO_D1/PC9)
- net MIC_VDD: now also C39.2, C9.2, MIC1.5 (VDD), MIC2.5 (VDD), TP17.1
- net at DD4.43 (OTG_ID/T1C3/RX1/PA10): now also XL3.2 (PM)
- net SX_RST: now reaches DD4.51 (SCK3/TX4/TX3/SDIO_D2/PC10)
- net SX_RST: now also DD1.7 (NRESET), TP1.1
- net NPX_PWR_EN: now reaches DD4.52 (MISO3/RX4/RX3/SDIO_D3/PC11)
- net NPX_PWR_EN: now also R16.2, Q4.1 (G)
- net NPX1_CTRL: now reaches DD4.53 (MOSI3/TX5/CK3/SDIO_CK/PC12)
- net NPX1_CTRL: now also DA3.2 (InA)
- net SX_NSS: now reaches DD4.54 (RX5/SDIO_CMD/PD2)
- net SX_NSS: now also DD1.19 (NSS), TP9.1
- net SX_SCK: now reaches DD4.55 (PB3/SCK1/SCK3/T2C2/SWO)
- net SX_SCK: now also DD1.16 (SCK), TP6.1
- net SX_MISO: now reaches DD4.56 (PB4/MISO1/MISO3/T3C1)
- net SX_MISO: now also DD1.17 (MISO)
- net SX_MOSI: now reaches DD4.57 (PB5/MOSI1/MOSI3/T3C2/CK1/LPTIM1_IN1)
- net SX_MOSI: now also DD1.18 (MOSI), TP8.1
- net PDM_IN6: now reaches DD4.61 (PB8/SDIO_D4/T4C3/T16C1/SCL1)
- net PDM_IN6: now also R6.1, TP14.1
- net SX_DIO0: now reaches DD4.62 (PB9/SDIO_D5/T4C4/T17C1/SDA1/IR_OUT)
- net SX_DIO0: now also DD1.8 (DIO0), TP2.1
- net ANT1: no longer names the net of L3.2
- net ANT1: now also C3.2, C7.1, L4.1; no longer C42.1
- net ANT2: no longer names the net of L3.1
- net ANT2: now also C4.1
- net Btn renamed Btn0
- net Btn0: now also XL2.2 (PM)
- net HP_OUTA: no longer names the net of DA1.15 (HP/LINE_OUTA)
- net HP_OUTA: no longer C14.2
- net HP_OUTB: no longer names the net of DA1.14 (HP/LINE_OUTB)
- net PWR_EN renamed AU_PWR_EN
- net SD_PWR: no longer names the net of Q1.3 (D)
- net SD_PWR: now also C42.1, DD2.8 (VCC)
- new net: C1.1, C2.1, DD1.25 (VR_PA), L1.1
- new net: C4.2, C6.1, L1.2, L2.2
- new net: Q2.4 (G), Q4.3 (D), Q5.1 (G), R14.2
- new net: MIC1.1 (DATA), R3.2
- new net: MIC2.1 (DATA), R6.2
- new net: MIC2.4 (CLK), R5.2
- new net: C31.1, DD1.2 (VR_ANA)
- new net: C3.1, C8.1, DA2.1 (RF1), L4.2
- new net: C17.1, DA2.3 (RF2)
- new net: C23.1, DA2.4 (CTRL), R4.2
- new net: C16.2, DA2.5 (RFC)
- new net: DD1.20 (RXTX/RF_MOD), R4.1
- new net: C17.2, C21.1, L6.2
- new net: C32.1, DD1.4 (VR_DIG)
- new net: MIC1.4 (CLK), R2.2
- new net: C16.1, C18.1, L5.1
- new net: ANT1.1 (RF), C19.1, L5.2
- new net: DD1.21 (RFI_HF), L6.1
- new net: DD1.27 (PA_BOOST), L2.1
- new net: C41.1, DD1.5 (XTA), XTAL1.1
- new net: C40.1, DD1.6 (XTB), XTAL1.2
- new net DIN0: DA3.4 (OutY), XL6.2 (PM)
- new net NPX_PWR: C48.2, DA3.5 (Vcc), Q2.5 (D), Q2.6 (D), Q2.7 (D), Q2.8 (D), Q5.3 (D), XL6.3
- new net PDM_IN2: DD4.35 (PB14/MISO2/SDA2/T15C1), R3.1, TP12.1
- no-connect marks 25 -> 31
Other:
- note added: "Accelerometers"
- note added: "Buffer"
- note added: "Button"
- note added: "Flash"
- note added: "I2C addr = 0x1C"
- note added: "Just GND"
- note added: "LORA radio"
- note added: "MCU"
- note added: "Maybe this one is acceptable: 50 mOhm"
- note added: "Mics"
- note added: "Neopixel"
- note added: "One or another"
- note removed: "Accelerometer I2C addr = 0x1C"
- note removed: "Balun"
- note removed: "CC Power Filter"
- note removed: "Headphones"
- note removed: "Keep CS High when sleeping"
- note removed: "Matching circuit"
- note removed: "Pins 15, 14, 11, 9, 4, 18"
- note removed: "Radio"
- moved on the sheet: B1, C10, C11, C12, C13, C20, C22, C25, C26, C33, C34, C35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

Commit message: Back to huge
Parts:
- removed B1: BAT, Installation:EEMB603030, symbol Power_kl:BAT
- removed C39, C42, C44, C45, C9: 0.1u, Capacitors:CAP_0603, symbol Tittar_kl:C
- removed C43: 10u, Capacitors:CAP_0603, symbol Tittar_kl:C
- removed DD2: W25Q128, SO_DIL_TSSOP:SO8_208MIL, symbol memory:W25Q32JV
- removed DD3: MMA8452Q, QFN_DFN:QFN16_5x3, symbol Sensors:MMA8452Q
- removed MIC1, MIC2: MSM261D3526Z1CM, Microphones:SPH0644, symbol Audio_kl:PDM_MIC_SPH0644
- removed Q1: IRLML6401, SOT:SOT23-3, symbol Transistors_kl:P_3PIN
- removed Q3: LED_5050, LEDs:LED_5050, symbol Tittar_kl:LED_5050
- removed R12, R13, R15: 1k, Resistors:RES_0603, symbol Tittar_kl:R
- removed R2, R3, R5, R6: 33R, Resistors:RES_0402_sm, symbol Tittar_kl:R
- removed R9: 100k, Resistors:RES_0603, symbol Tittar_kl:R
- removed TP10, TP12, TP14, TP17: TESTPOINT, PCB:TESTPOINT_1MM, symbol pcb_details:TESTPOINT
- removed XL2: CONN_2, Connectors:W02_Pitch_2d54, symbol Connectors_kl:CONN_2
- added C? (x2): 0.1u, Capacitors:CAP_0402, symbol Tittar_kl:C
- added C? (x2): 10u, Capacitors:CAP_0603, symbol Tittar_kl:C
- added C? (x2): 1u, Capacitors:CAP_0603, symbol Tittar_kl:C
- added C?: 0.1u, Capacitors:CAP_0603, symbol Tittar_kl:C
- added DD? (x2): ICN2595, SO_DIL_TSSOP:TSSOP24_150_0635, symbol LED_Driver:ICN2595
- added F?: Fuse0R, Resistors:RES_0603_FUSE, symbol Tittar_kl:Fuse0R
- added Q? (x10): LED_5050, LEDs:LED_5050, symbol Tittar_kl:LED_5050
- added R? (x2): 3k, Resistors:RES_0402_sm, symbol Tittar_kl:R
- added R?: 2k, Resistors:RES_0603, symbol Tittar_kl:R
- added R?: 100k, Resistors:RES_0603, symbol Tittar_kl:R
- added RP? (x2): REFPOINT, PCB:REF_POINT_1MM, symbol pcb_details:REFPOINT
- added XL?: CONN_2, Connectors:SLD_2_2D5_1mm, symbol Connectors_kl:CONN_2
- added XL?: CONN_2, Connectors:WB-02R(MW-2MR), symbol Connectors_kl:CONN_2
Connections:
- net +BATT: now also F?.1, XL?.2 (PM)
- net Btn0: no longer DD4.14 (ADC12-5/WKUP1/T2C1/T5C1/TX4/PA0)
- net GND: now also C?.1, C?.1, C?.1, C?.1, C?.2, C?.2, DD?.1 (GND), DD?.1 (GND), R?.1, R?.2, R?.2, XL?.1 (P1), XL?.2 (PM)
- net PWR_UNST_ALWAYS: now also F?.2
- net SX_DIO1: no longer DD4.15 (ADC12-6/T2C2/T5C2/RX4/PA1)
- net SX_DIO2: no longer DD4.16 (ADC12-7/WKUP4/T15C1/T2C3/T5C3/TX2/PA2)
- net SX_DIO3: no longer DD4.17 (ADC12-8/T15C2/T2C4/T5C4/RX2/PA3)
- net SX_RST: now also DD4.37 (T3C1/T8C1/SDIO_D6/PC6); no longer DD4.51 (SCK3/TX4/TX3/SDIO_D2/PC10)
- net at DD4.24 (ADC12-13/TX3/PC4): no longer XL3.3
- net at DD4.25 (ADC12-14/RX3/PC5): no longer XL3.4
- net at DD4.43 (OTG_ID/T1C3/RX1/PA10): no longer XL3.2 (PM)
- net MICBIAS: now reaches DA1.20 (MICBIAS)
- net MICBIAS: now also C?.1, R?.2
- net MIC1+: now reaches DA1.21 (AIN4A/MIC1+)
- net MIC1+: now also C?.1
- net MIC1-: now reaches DA1.23 (AIN3A/MIC1-)
- net MIC1-: now also C?.1
- net AU_SDOUT: now reaches DA1.36 (SDOUT)
- net MEM_PWR_EN: no longer names the net of DD4.28 (PB2/LPTIM1_OUT/RTC_OUT)
- net MIC_VDD: no longer names the net of DD4.40 (OTG_NOE/T3C4/T8C4/SDIO_D1/PC9)
- net PDM_CLK: no longer names the net of DD4.10 (ADC123-3/LPTIM1_IN2/MISO2/PC2)
- net PDM_IN2: no longer names the net of DD4.35 (PB14/MISO2/SDA2/T15C1)
- net PDM_IN6: no longer names the net of DD4.61 (PB8/SDIO_D4/T4C3/T16C1/SCL1)
- net QSPI_CLK: no longer names the net of DD4.29 (PB10/T2C3/SCK2/SCL2/TX3/LPRX1/QSPI_CLK)
- net QSPI_IO0: no longer names the net of DD4.27 (PB1/T3C4/QSPI0/LPTIM2_IN1/ADC12-16)
- net QSPI_IO1: no longer names the net of DD4.26 (PB0/T3C3/QSPI1/ADC12-15)
- net QSPI_IO2: no longer names the net of DD4.23 (ADC12-12/T3C2/T17C1/QSPI2/MOSI1/PA7)
- net QSPI_IO3: no longer names the net of DD4.22 (ADC12-11/T3C1/T16C1/QSPI3/MISO1/PA6)
- net QSPI_NCS: no longer names the net of DD4.30 (PB11/T2C4/SDA2/RX3/LPTX1/QSPI_NCS)
- new net: DD?.12 (Y7), Q?.4 (B)
- new net: DD?.11 (Y6), Q?.5 (G)
- new net: DD?.10 (Y5), Q?.6
- new net: DD?.15 (Y10), Q?.4 (B)
- new net: DD?.14 (Y9), Q?.5 (G)
- new net: DD?.13 (Y8), Q?.6
- new net: DD?.23 (R-EXT), R?.1 (x2)
- new net: DD?.6 (Y1), Q?.4 (B)
- new net: DD?.5 (Y0), Q?.5 (G)
- new net: DD?.20 (Y15), Q?.6
- new net: C?.2, R?.1, R?.2, XL?.1 (P1)
- new net: DD?.18 (Y13), Q?.4 (B)
- new net: DD?.17 (Y12), Q?.5 (G)
- new net: DD?.16 (Y11), Q?.6
- new net: DD?.10 (Y5), Q?.4 (B)
- new net: DD?.9 (Y4), Q?.5 (G)
- new net: DD?.8 (Y3), Q?.6
- new net: DD?.13 (Y8), Q?.4 (B)
- new net: DD?.12 (Y7), Q?.5 (G)
- new net: DD?.11 (Y6), Q?.6
- new net: DD?.2 (DataIn), DD?.22 (DataOut)
- new net: DD?.7 (Y2), Q?.6
- new net: DD?.8 (Y3), Q?.5 (G)
- new net: DD?.9 (Y4), Q?.4 (B)
- new net: DD?.14 (Y9), Q?.6
- new net: DD?.15 (Y10), Q?.5 (G)
- new net: DD?.16 (Y11), Q?.4 (B)
- new net: DD?.17 (Y12), Q?.6
- new net: DD?.18 (Y13), Q?.5 (G)
- new net: DD?.19 (Y14), Q?.4 (B)
- new net: DD?.5 (Y0), Q?.6
- new net: DD?.6 (Y1), Q?.5 (G)
- new net: DD?.7 (Y2), Q?.4 (B)
- new net LED_CLK: DD?.3 (CLK), DD?.3 (CLK)
- new net LED_DATA: DD?.2 (DataIn)
- new net LED_LATCH: DD?.4 (Latch), DD?.4 (Latch)
- new net LED_OUT_EN: DD?.21 (~OutEn), DD?.21 (~OutEn)
- new net PWR_LEDS: C?.2, C?.2, C?.2, C?.2, DD?.24 (VCC), DD?.24 (VCC), Q?.1, Q?.1, Q?.1, Q?.1, Q?.1, Q?.1, Q?.1, Q?.1, Q?.1, Q?.1, Q?.2, Q?.2, Q?.2, Q?.2, Q?.2, Q?.2, Q?.2, Q?.2, Q?.2, Q?.2, Q?.3, Q?.3, Q?.3, Q?.3, Q?.3, Q?.3, Q?.3, Q?.3, Q?.3, Q?.3
- no-connect marks 31 -> 29
Other:
- note added: "Accelerometer"
- note added: "Mic1"
- note added: "Put 0R If charger is not required"
- note removed: "Accelerometers"
- note removed: "Button"
- note removed: "Flash"
- note removed: "I2C addr = 0x1C"
- note removed: "Mics"
- note removed: "One or another"
- moved on the sheet: ANT1, C1, C10, C11, C12, C13, C14, C15, C16, C17, C18, C19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

Commit message: + PCB is ready
Parts:
- removed C61, C62: 10u, Capacitors:CAP_0603, symbol Tittar_kl:C
- removed DA4: TP4056, SO_DIL_TSSOP:SO8_150MIL, symbol Power_kl:TP4056
- removed Q2: IRF9317, SO_DIL_TSSOP:SO8_150MIL, symbol Transistors_kl:P_8PIN
- removed Q6: IRLML6401, SOT:SOT23-3, symbol Transistors_kl:P_3PIN
- removed Q8: 2N7002, SOT:SOT23-3, symbol Transistors_kl:N_3PIN
- removed R18, R24: 100k, Resistors:RES_0603, symbol Tittar_kl:R
- removed R21: 10k, Resistors:RES_0603, symbol Tittar_kl:R
- removed R22: 1.2k, Resistors:RES_0603, symbol Tittar_kl:R
- removed XL3: CONN_4, Connectors:PLS-4, symbol Connectors_kl:CONN_4
- removed XL4: CONN_6, Connectors:PLS-6, symbol Connectors_kl:CONN_6
- removed XL6: CONN_3, Connectors:SLD_3_2D5, symbol Connectors_kl:CONN_3
- added C17: 10u, Capacitors:CAP_0603_Silks, symbol Tittar_kl:C
- added C18, C20, C38, C67, C68: 0.1u, Capacitors:CAP_0603_Silks, symbol Tittar_kl:C
- added C19: 1u, Capacitors:CAP_0603_Silks, symbol Tittar_kl:C
- added DD2: STM32G070CxTx, LQFP_TQFP:LQFP48, symbol st_kl:STM32G070CxTx
- added HOLE5, HOLE6: HOLE_METALLED, PCB:Hole3d5_out10mm, symbol pcb_details:HOLE_METALLED
- added HOLE7, HOLE8, HOLE9: HOLE_METALLED, PCB:Hole3d3_out5d5mm, symbol pcb_details:HOLE_METALLED
- added L9: BLM15AG102, Inductors:IND_0402, symbol Tittar_kl:L
- added Q1: IRLML6401, SOT:SOT23-3, symbol Transistors_kl:P_3PIN
- added R10: 100k, Resistors:RES_0603, symbol Tittar_kl:R
- added R16, R17: 10k, Resistors:RES_0603, symbol Tittar_kl:R
- added R6, R7: 4k7, Resistors:RES_0603, symbol Tittar_kl:R
- added RP3, RP4: REFPOINT, PCB:REF_POINT_2MM, symbol pcb_details:REFPOINT
- added SW1, SW2, SW3: BUTTON, BtnsSwitches:BTN_4x4_SMD, symbol BtnsSwitches:BUTTON
- added TP3: TESTPOINT, PCB:TESTPOINT_1MM, symbol pcb_details:TESTPOINT
- added XL1: PLS-6, Connectors:PLS-6_LOCK, symbol Connectors_kl:CONN_6
- added XL12: CONN_2, Connectors:SLD_2_2D5_1mm, symbol Connectors_kl:CONN_2
- added XL4: PLS1, Connectors:PLS-1Rnd, symbol Connectors_kl:CONN_1
- added XL7: CONN_MICROSD, Installation:MICROSD_CAP_FIX05A, symbol Connectors_kl:CONN_MICROSD
- added XL9: CONN_3, Connectors:SLD_3_2D5, symbol Connectors_kl:CONN_3
- ANT1: footprint Antennas:ANT_868_IFA_SIMPLEJOY -> Antennas:ANT_IFA_MUSHROOM
- C1: renamed from C5; footprint Capacitors:CAP_0603 -> Capacitors:CAP_0603_Silks
- C10: renamed from C20; footprint Capacitors:CAP_0603 -> Capacitors:CAP_0603_Silks
- C11: renamed from C22; footprint Capacitors:CAP_0603 -> Capacitors:CAP_0603_Silks
- C12: renamed from C47; footprint Capacitors:CAP_0603 -> Capacitors:CAP_0603_Silks
- C13: renamed from C25; footprint Capacitors:CAP_0603 -> Capacitors:CAP_0603_Silks
- C14, C37, C39, C61, C63: renamed from C?; footprint Capacitors:CAP_0603 -> Capacitors:CAP_0603_Silks
- C15: renamed from C26; footprint Capacitors:CAP_0603 -> Capacitors:CAP_0603_Silks
- C16: renamed from C33; footprint Capacitors:CAP_0603 -> Capacitors:CAP_0603_Silks
- C2: renamed from C10; footprint Capacitors:CAP_0603 -> Capacitors:CAP_0603_Silks
- C21: renamed from C34; footprint Capacitors:CAP_0603 -> Capacitors:CAP_0603_Silks
- C22: renamed from C35; footprint Capacitors:CAP_0603 -> Capacitors:CAP_0603_Silks
- C23: renamed from C36; footprint Capacitors:CAP_0603 -> Capacitors:CAP_0603_Silks
- C24: renamed from C37; footprint Capacitors:CAP_0603 -> Capacitors:CAP_0603_Silks
- C25: renamed from C38; footprint Capacitors:CAP_0603 -> Capacitors:CAP_0603_Silks
- C26: renamed from C49; footprint Capacitors:CAP_0603 -> Capacitors:CAP_0603_Silks
- C27: renamed from C50; footprint Capacitors:CAP_0603 -> Capacitors:CAP_0603_Silks
- C28: renamed from C52; footprint Capacitors:CAP_0603 -> Capacitors:CAP_0603_Silks
- C29: renamed from C53; footprint Capacitors:CAP_0603 -> Capacitors:CAP_0603_Silks
- C3: renamed from C11; footprint Capacitors:CAP_0603 -> Capacitors:CAP_0603_Silks
- C30: renamed from C54; footprint Capacitors:CAP_0603 -> Capacitors:CAP_0603_Silks
- C31: renamed from C55; footprint Capacitors:CAP_0603 -> Capacitors:CAP_0603_Silks
- C32: renamed from C56; footprint Capacitors:CAP_0603 -> Capacitors:CAP_0603_Silks
- C33: renamed from C57; footprint Capacitors:CAP_0603 -> Capacitors:CAP_0603_Silks
- C34: renamed from C58; footprint Capacitors:CAP_0603 -> Capacitors:CAP_0603_Silks
- C35: renamed from C59; footprint Capacitors:CAP_0603 -> Capacitors:CAP_0603_Silks
- C36: renamed from C60; footprint Capacitors:CAP_0603 -> Capacitors:CAP_0603_Silks
- C4: renamed from C12; footprint Capacitors:CAP_0603 -> Capacitors:CAP_0603_Silks
- C48: renamed from C16; value 47pFpF -> 47pF
- C5: renamed from C13; footprint Capacitors:CAP_0603 -> Capacitors:CAP_0603_Silks
- C6: renamed from C14; footprint Capacitors:CAP_0603 -> Capacitors:CAP_0603_Silks
- C62, C64: renamed from C?; footprint Capacitors:CAP_0402 -> Capacitors:CAP_0603_Silks
- C69: renamed from C63; footprint Capacitors:CAP_0603 -> Capacitors:CAP_0603_Silks
- C7: renamed from C15; footprint Capacitors:CAP_0603 -> Capacitors:CAP_0603_Silks
- C70: renamed from C64; footprint Capacitors:CAP_0603 -> Capacitors:CAP_0603_Silks
- C71: renamed from C65; footprint Capacitors:CAP_0603 -> Capacitors:CAP_0603_Silks
- C72: renamed from C66; footprint Capacitors:CAP_0603 -> Capacitors:CAP_0603_Silks
- C8: renamed from C51; footprint Capacitors:CAP_0603 -> Capacitors:CAP_0603_Silks
- C9: renamed from C46; footprint Capacitors:CAP_0603 -> Capacitors:CAP_0603_Silks
- DD3: renamed from DD5; footprint (none) -> LGA:LGA16_3X3_5_3
- HOLE1, HOLE2, HOLE3, HOLE4: footprint PCB:Hole2d4_out4d5mm -> PCB:Hole3d5_out10mm
- L1: renamed from L8; value BLM15 -> BLM15AG102
- L8: renamed from L7; value Choke -> BLM15AG102
- Logo1: footprint Pictures:Ostranna_12d7_10d1 -> Pictures:Ostranna_16d9_13d5
- R14, R15: renamed from R?; footprint Resistors:RES_0402_sm -> Resistors:RES_0603
- R19: value 0R2 -> 10k; footprint Resistors:RES_1206 -> Resistors:RES_0603
- RP1, RP2: renamed from RP?; footprint PCB:REF_POINT_1MM -> PCB:REF_POINT_2MM
- XL6: renamed from XL5; footprint Connectors:USBmicro_MOLEX_WM17142 -> Connectors:USBmicro_MOLEX_1050170001
- XL8: renamed from XL?; footprint Connectors:WB-02R(MW-2MR) -> Connectors:WB-02(MW-2M)LongContacts
- XTAL1: renamed from XTAL2; footprint Quartz:0503x4-4 -> Quartz:03225C4
- gave numbers to parts that had none: 16
- renumbered C48 to C40, C1 to C41, C2 to C42, C3 to C43, C4 to C44, C6 to C45, C7 to C46, C8 to C47, C17 to C49, C18 to C50, C19 to C51, C21 to C52, C23 to C53, C24 to C54, C27 to C55, C28 to C56, C29 to C57, C30 to C58, C31 to C59, C32 to C60, C40 to C65, C41 to C66, DA3 to DA2, DA2 to DA3, DD4 to DD1, DD1 to DD6, L1 to L2, L2 to L3, L3 to L4, L4 to L5, L5 to L6, L6 to L7, Q4 to Q13, Q7 to Q15, Q5 to Q2, R14 to R11, R16 to R12, R4 to R13, R17 to R18, R10 to R2, R20 to R21, R23 to R24, R11 to R3, R7 to R4, R8 to R5, TP11 to TP1, TP5 to TP10, TP6 to TP11, TP7 to TP12, TP8 to TP13, TP9 to TP14, TP13 to TP2, TP15 to TP4, TP16 to TP5, TP1 to TP6, TP2 to TP7, TP3 to TP8, TP4 to TP9, XL7 to XL11, XL1 to XL3, XTAL1 to XTAL2
Connections:
- net 5V_MID is gone; now on net BTN0: R19.2
- net MEASURE_EN is gone; now on net LED_CLK: DD1.21 (ADC12-10/T2C1/DAC2/SCK1/PA5)
- net PWR_LEDS is gone; now on net PwrUnst: C61.2, C62.2, C63.2, C64.2, DD4.24 (VCC), DD5.24 (VCC), Q10.1, Q10.2, Q10.3, Q11.1, Q11.2, Q11.3, Q12.1, Q12.2, Q12.3, Q3.1, Q3.2, Q3.3, Q4.1, Q4.2, Q4.3, Q5.1, Q5.2, Q5.3, Q6.1, Q6.2, Q6.3, Q7.1, Q7.2, Q7.3, Q8.1, Q8.2, Q8.3, Q9.1, Q9.2, Q9.3
- net +3v3: now also L9.2, Q1.2 (S), R10.1, SW1.2, SW2.2, SW3.2, XL1.1
- net +5v: no longer R19.1
- net ACC_INT1: now also DD2.1 (WKUP2/PC13)
- net AU_LRCK: now also DD1.62 (PB9/SDIO_D5/T4C4/T17C1/SDA1/IR_OUT); no longer DD1.33 (PB12/CK3)
- net AU_RST: now also DA6.3 (EN), DD1.10 (ADC123-3/LPTIM1_IN2/MISO2/PC2); no longer DD1.11 (ADC123-4/MOSI2/PC3)
- net AU_SCLK: now also DD1.29 (PB10/T2C3/SCK2/SCL2/TX3/LPRX1/QSPI_CLK); no longer DD1.34 (PB13/SCK2/SCL2)
- net AU_SDIN: now also DD1.11 (ADC123-4/MOSI2/PC3); no longer DD1.36 (PB15/MOSI2/T15C2)
- net AU_SDOUT: now also DD1.57 (PB5/MOSI1/MOSI3/T3C2/CK1/LPTIM1_IN1), TP3.1
- net BAT_MEAS: now also DD1.24 (ADC12-13/TX3/PC4), DD2.15 (ADC4/NSS1/MOSI2/T14C1/PA4); no longer DD1.20 (ADC12-9/LPTIM2_OUT/DAC1/CK2/PA4)
- net DIN0: now also XL9.2 (PM)
- net GND: now also R19.1, R21.2, C17.1, C18.1, C19.1, C20.1, C38.2, C67.1, C68.1, DD2.7 (VSS/VSSA), HOLE5.H, HOLE6.H, HOLE7.H, HOLE8.H, HOLE9.H, R17.1, XL1.3, XL7.6 (GND), XL7.H (Housing), XL9.1 (P1)
- net LED_CLK: now also DD1.22 (ADC12-11/T3C1/T16C1/QSPI3/MISO1/PA6), DD2.42 (PB3/SCK1/T1C2), DD2.43 (PB4/MISO1/T3C1)
- net LED_DATA: now also DA2.2 (InA), DD1.23 (ADC12-12/T3C2/T17C1/QSPI2/MOSI1/PA7), DD2.44 (PB5/MOSI1/T3C2)
- net LED_LATCH: now also DD1.27 (PB1/T3C4/QSPI0/LPTIM2_IN1/ADC12-16), DD2.20 (PB1/T14C1/T3C4/ADC9)
- net LED_OUT_EN: now also DD1.17 (ADC12-8/T15C2/T2C4/T5C4/RX2/PA3), DD2.18 (ADC7/MOSI1/T3C2/T14C1/T17C1/PA7), R16.2
- net NPX_PWR: now also XL9.3
- net NPX_PWR_EN: now also DD1.37 (T3C1/T8C1/SDIO_D6/PC6), DD2.45 (PB6/TX1/T1C3/MISO2/SCL1); no longer DD1.52 (MISO3/RX4/RX3/SDIO_D3/PC11)
- net PwrMCU: now also C17.2, C18.2, C19.2, C20.2, DD2.4 (VBAT), DD2.5 (VREF+), DD2.6 (VDD/VDDA), L9.1, R6.2, R7.2
- net PwrUnst: now also C3.1, C4.1, C5.1, C6.1, C7.1, C71.1, DA1.5 (VP), DA1.8 (VP), DA6.1 (IN), R16.1
- net SPK_M: now also XL12.2 (PM)
- net SPK_P: now also XL12.1 (P1)
- net SWCLK: now also DD2.36 (BOOT0/TX2/SWCLK/PA14), XL1.2
- net SWDIO: now also DD2.35 (IROUT/SWDIO/PA13), XL1.4
- net SX_DIO0: now also DD1.26 (PB0/T3C3/QSPI1/ADC12-15), DD2.47 (PB8/SCK2/T16C1/TX3/SCL1); no longer DD1.62 (PB9/SDIO_D5/T4C4/T17C1/SDA1/IR_OUT)
- net SX_DIO1: now also DD1.28 (PB2/LPTIM1_OUT/RTC_OUT), DD2.48 (PB9/IR_OUT/T17C1/RX3/NSS2/SDA1)
- net SX_DIO2: now also DD1.55 (PB3/SCK1/SCK3/T2C2/SWO), DD2.22 (PB10/TX3/SCK2/SCL2/ADC11)
- net SX_DIO3: now also DD1.56 (PB4/MISO1/MISO3/T3C1), DD2.23 (PB11/MOSI2/RX3/SDA2/ADC15)
- net SX_MISO: now also DD1.35 (PB14/MISO2/SDA2/T15C1), DD2.26 (PB14/MISO2/T15C1/SDA2); no longer DD1.56 (PB4/MISO1/MISO3/T3C1)
- net SX_MOSI: now also DD1.36 (PB15/MOSI2/T15C2), DD2.27 (PB15/MOSI2/T15C2); no longer DD1.57 (PB5/MOSI1/MOSI3/T3C2/CK1/LPTIM1_IN1)
- net SX_NSS: now also DD1.33 (PB12/CK3), DD2.24 (PB12/NSS2/ADC16); no longer DD1.54 (RX5/SDIO_CMD/PD2)
- net SX_RST: now also DD1.61 (PB8/SDIO_D4/T4C3/T16C1/SCL1), DD2.46 (PB7/RX1/MOSI2/SDA1); no longer DD1.37 (T3C1/T8C1/SDIO_D6/PC6)
- net SX_SCK: now also DD1.34 (PB13/SCK2/SCL2), DD2.25 (PB13/SCK2/SCL2); no longer DD1.55 (PB3/SCK1/SCK3/T2C2/SWO)
- net UART_RX: now also DD1.43 (OTG_ID/T1C3/RX1/PA10), DD2.32 (MOSI2/RX1/T1C3/SDA1/PA10), XL1.6; no longer DD1.59 (PB7/SDA1/T4C2/RX1/LPTIM1_IN2)
- net UART_TX: now also DD1.42 (OTG_VBUS/T1C2/TX1/PA9), DD2.29 (MCO/TX1/T1C2/MISO2/SCL1/PA9), XL1.5; no longer DD1.58 (PB6/SCL1/T4C1/TX1)
- net BTN0: now reaches DD1.14 (ADC12-5/WKUP1/T2C1/T5C1/TX4/PA0)
- net BTN0: now also C67.2, C68.2, DD2.11 (ADC0/WKUP1/SCK2/TX4/PA0), R17.2, SW1.1, SW2.1, SW3.1
- net DBG_PIN: now reaches DD1.30 (PB11/T2C4/SDA2/RX3/LPTX1/QSPI_NCS)
- net DBG_PIN: now also DD2.19 (PB0/NSS1/T3C2/RX3/ADC8), XL4.1 (P1)
- net SD_PWR_EN: now reaches DD1.38 (T3C2/T8C2/SDIO_D7/PC7)
- net SD_PWR_EN: now also Q1.1 (G), R10.2
- net SD_DAT0: now reaches DD1.39 (T3C3/T8C3/SDIO_D0/PC8)
- net SD_DAT0: now also XL7.7 (MISO/DAT0)
- net SD_DAT1: now reaches DD1.40 (OTG_NOE/T3C4/T8C4/SDIO_D1/PC9)
- net SD_DAT1: now also XL7.8 (DAT1)
- net at R2.1: now also DD1.20 (ADC12-9/LPTIM2_OUT/DAC1/CK2/PA4); no longer DD1.42 (OTG_VBUS/T1C2/TX1/PA9)
- net SD_DAT2: now reaches DD1.51 (SCK3/TX4/TX3/SDIO_D2/PC10)
- net SD_DAT2: now also XL7.1 (DAT2)
- removed net AU_PWR: C3.1, C4.1, C5.1, C6.1, C7.1, C71.1, DA1.5 (VP), DA1.8 (VP), DA6.1 (IN), DA6.3 (EN)
- net ChrgEn: no longer names the net of DD1.4 (OC32OUT/PC15)
- net IsCharging: no longer names the net of DD1.3 (OC32IN/PC14)
- net NPX1_CTRL renamed SD_CLK
- net SD_CLK: now also XL7.5 (SCK/CLK); no longer DA2.2 (InA)
- net SCL renamed AU_SCL
- net AU_SCL: no longer DD3.4 (SCL(SPC))
- net SDA renamed AU_SDA
- net AU_SDA: no longer DD3.6 (SDA(SDI/SDO))
- new net I2C_SCL: DD1.58 (PB6/SCL1/T4C1/TX1), DD2.33 (MISO1/T1C4/SCL2/PA9/PA11), DD3.4 (SCL(SPC)), R6.1
- new net I2C_SDA: DD1.59 (PB7/SDA1/T4C2/RX1/LPTIM1_IN2), DD2.34 (MOSI1/SDA2/PA12), DD3.6 (SDA(SDI/SDO)), R7.1
- new net SD_CMD: DD1.54 (RX5/SDIO_CMD/PD2), XL7.3 (MOSI/CMD)
- new net SD_DAT3: DD1.52 (MISO3/RX4/RX3/SDIO_D3/PC11), XL7.2 (~SS~/DAT3)
- new net SD_PWR: C38.1, Q1.3 (D), XL7.4 (VDD)
- no-connect marks 29 -> 52
Other:
- note added: "Buttons"
- note added: "Latch generated by TIM3 C4"
- note added: "MCU Heavy"
- note added: "MCU Lite"
- note added: "SCK1 is connected with T3C1 TIM3 counts SPI pulses"
- note removed: "Charger 1.2k => 1000mA"
- note removed: "Just pins"
- note removed: "MCU"
- note removed: "Maybe this one is acceptable: 50 mOhm"
- moved on the sheet: ANT1, C1, C10, C11, C12, C13, C14, C15, C16, C2, C21, C22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

Commit message: + Leds are ok
Parts:
- C17, C18, C19, C20, C67, DD2, L9, R17: Variant (none) -> 1
- C26, C27, C61, C62, C63, C64, C69, C70, DA5, DD3, DD4, DD5, Q10, Q11, Q12, Q3, Q4, Q5, Q6, Q7, Q8, Q9, R14, R15, R16, R18, R21, R6, R7, SW1, SW2, SW3: Variant (none) -> all
- F1, HOLE1, HOLE2, HOLE3, HOLE4, HOLE5, HOLE6, HOLE7, HOLE8, HOLE9, Logo1, XL10: DoNotBOM (none) -> true
