File: Floe_hw/Floe.kicad_sch (KiCad schematic)
At the start: 174 parts, among them Q1 IRLML6401, Q10 LED_5050, Q11 LED_5050, Q12 LED_5050, Q13 2N7002, Q15 IRLML6401, Q2 IRLML6401, Q3 LED_5050, Q4 LED_5050, Q5 LED_5050, Q6 LED_5050, Q7 LED_5050, Q8 LED_5050, Q9 LED_5050, SW1 BUTTON, SW2 BUTTON, SW3 BUTTON

Commit message: Algo2
Parts:
- added C?: 2.2pF, Capacitors:CAP_0402, symbol Tittar_kl:C
- added L?: 4.7nH, Inductors:IND_0402, symbol Tittar_kl:L
Connections:
- net GND: now also L?.2
- new net: C?.2, L?.1
Changed lines of the file:
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@@
   (junction (at 510.54 165.1) (diameter 1.016) (color 0 0 0 0))
   (junction (at 510.54 167.64) (diameter 1.016) (color 0 0 0 0))
+  (junction (at 515.62 233.68) (diameter 1.016) (color 0 0 0 0))
   (junction (at 515.62 259.08) (diameter 1.016) (color 0 0 0 0))
   (junction (at 516.89 165.1) (diameter 1.016) (color 0 0 0 0))
@@
   (junction (at 552.45 365.76) (diameter 1.016) (color 0 0 0 0))
   (junction (at 556.26 45.72) (diameter 1.016) (color 0 0 0 0))
-  (no_connect (at 547.37 101.6))
-  (no_connect (at 547.37 48.26))
+  (no_connect (at 212.09 368.3))
+  (no_connect (at 547.37 58.42))
+  (no_connect (at 242.57 106.68))
+  (no_connect (at 547.37 91.44))
+  (no_connect (at 149.86 52.07))
+  (no_connect (at 396.24 245.11))
   (no_connect (at 547.37 53.34))
-  (no_connect (at 336.55 36.83))
-  (no_connect (at 547.37 60.96))
-  (no_connect (at 508 156.21))
+  (no_connect (at 293.37 74.93))
   (no_connect (at 450.85 92.71))
-  (no_connect (at 547.37 93.98))
-  (no_connect (at 450.85 95.25))
-  (no_connect (at 547.37 66.04))
-  (no_connect (at 293.37 85.09))
-  (no_connect (at 293.37 90.17))
-  (no_connect (at 149.86 134.62))
-  (no_connect (at 149.86 49.53))
-  (no_connect (at 547.37 91.44))
   (no_connect (at 173.99 257.81))
-  (no_connect (at 547.37 104.14))
-  (no_connect (at 234.95 106.68))
-  (no_connect (at 547.37 111.76))
+  (no_connect (at 48.26 109.22))
   (no_connect (at 547.37 50.8))
-  (no_connect (at 171.45 257.81))
-  (no_connect (at 396.24 245.11))
-  (no_connect (at 450.85 50.8))
-  (no_connect (at 547.37 88.9))
-  (no_connect (at 149.86 132.08))
-  (no_connect (at 336.55 39.37))
-  (no_connect (at 547.37 83.82))
-  (no_connect (at 474.98 170.18))
+  (no_connect (at 293.37 80.01))
+  (no_connect (at 547.37 109.22))
   (no_connect (at 237.49 106.68))
-  (no_connect (at 240.03 106.68))
-  (no_connect (at 356.87 247.65))
   (no_connect (at 149.86 102.87))
-  (no_connect (at 293.37 72.39))
-  (no_connect (at 293.37 80.01))
-  (no_connect (at 48.26 109.22))
-  (no_connect (at 293.37 77.47))
-  (no_connect (at 547.37 58.42))
-  (no_connect (at 149.86 85.09))
   (no_connect (at 396.24 266.7))
-  (no_connect (at 547.37 109.22))
-  (no_connect (at 149.86 52.07))
-  (no_connect (at 508 158.75))
-  (no_connect (at 396.24 247.65))
-  (no_connect (at 293.37 74.93))
-  (no_connect (at 356.87 245.11))
-  (no_connect (at 140.97 285.75))
+  (no_connect (at 149.86 85.09))
+  (no_connect (at 149.86 49.53))
+  (no_connect (at 171.45 257.81))
+  (no_connect (at 240.03 106.68))
+  (no_connect (at 508 156.21))
   (no_connect (at 547.37 96.52))
-  (no_connect (at 212.09 368.3))
-  (no_connect (at 242.57 106.68))
+  (no_connect (at 547.37 66.04))
+  (no_connect (at 293.37 77.47))
+  (no_connect (at 140.97 285.75))
+  (no_connect (at 547.37 111.76))
   (no_connect (at 336.55 54.61))
-  (no_connect (at 508 161.29))
+  (no_connect (at 149.86 134.62))
+  (no_connect (at 336.55 36.83))
+  (no_connect (at 293.37 72.39))
+  (no_connect (at 547.37 83.82))
+  (no_connect (at 508 158.75))
+  (no_connect (at 547.37 104.14))
+  (no_connect (at 547.37 101.6))
+  (no_connect (at 293.37 90.17))
   (no_connect (at 450.85 88.9))
+  (no_connect (at 293.37 85.09))
+  (no_connect (at 547.37 93.98))
+  (no_connect (at 149.86 132.08))
+  (no_connect (at 547.37 60.96))
+  (no_connect (at 336.55 39.37))
+  (no_connect (at 356.87 247.65))
+  (no_connect (at 474.98 170.18))
+  (no_connect (at 234.95 106.68))
+  (no_connect (at 450.85 95.25))
+  (no_connect (at 547.37 88.9))
+  (no_connect (at 547.37 48.26))
+  (no_connect (at 450.85 50.8))
+  (no_connect (at 396.24 247.65))
+  (no_connect (at 508 161.29))
+  (no_connect (at 356.87 245.11))
   (wire (pts (xy 16.51 91.44) (xy 17.78 91.44))
     (stroke (width 0) (type solid) (color 0 0 0 0))
@@
     (stroke (width 0) (type solid) (color 0 0 0 0))
   )
+  (wire (pts (xy 509.27 233.68) (xy 515.62 233.68))
+    (stroke (width 0) (type solid) (color 0 0 0 0))
+  )
   (wire (pts (xy 509.27 259.08) (xy 515.62 259.08))
     (stroke (width 0) (type solid) (color 0 0 0 0))
@@
     (stroke (width 0) (type solid) (color 0 0 0 0))
   )
+  (wire (pts (xy 515.62 233.68) (xy 518.16 233.68))
+    (stroke (width 0) (type solid) (color 0 0 0 0))
+  )
+  (wire (pts (xy 515.62 237.49) (xy 515.62 233.68))
+    (stroke (width 0) (type solid) (color 0 0 0 0))
+  )
+  (wire (pts (xy 515.62 247.65) (xy 515.62 250.19))
+    (stroke (width 0) (type solid) (color 0 0 0 0))
+  )
   (wire (pts (xy 515.62 259.08) (xy 518.16 259.08))
     (stroke (width 0) (type solid) (color 0 0 0 0))
@@
     (stroke (width 0) (type solid) (color 0 0 0 0))
   )
+  (wire (pts (xy 528.32 233.68) (xy 534.67 233.68))
+    (stroke (width 0) (type solid) (color 0 0 0 0))
+  )
   (wire (pts (xy 528.32 259.08) (xy 530.86 259.08))
     (stroke (width 0) (type solid) (color 0 0 0 0))
@@
     )
   )
+  (symbol (lib_id "power:GND") (at 515.62 250.19 0) (unit 1)
+    (in_bom yes) (on_board yes)
+    (property "Reference" "#PWR?" (id 0) (at 517.906 250.698 0)
+      (effects (font (size 0.762 0.762)) hide)
+    )
+    (property "Value" "GND" (id 1) (at 515.62 252.222 0)
+      (effects (font (size 0.762 0.762)) hide)
+    )
+    (property "Footprint" "" (id 2) (at 515.62 250.19 0)
+      (effects (font (size 1.524 1.524)) hide)
+    )
+    (property "Datasheet" "" (id 3) (at 515.62 250.19 0)
+      (effects (font (size 1.524 1.524)) hide)
+    )
+  )
   (symbol (lib_id "power:GND") (at 515.62 273.05 0) (unit 1)
     (in_bom yes) (on_board yes)
@@
     )
   )
+  (symbol (lib_id "Tittar_kl:L") (at 515.62 242.57 0) (unit 1)
+    (in_bom yes) (on_board yes)
+    (property "Reference" "L?" (id 0) (at 518.5664 242.57 90))
+    (property "Value" "4.7nH" (id 1) (at 513.715 242.57 90))
+    (property "Footprint" "Inductors:IND_0402" (id 2) (at 517.144 242.316 90)
+      (effects (font (size 1.016 1.016)) hide)
+    )
+    (property "Datasheet" "" (id 3) (at 513.08 246.126 90)
+      (effects (font (size 1.524 1.524)) hide)
+    )
+    (property "Price" "4" (id 4) (at 515.62 243.586 90)
+      (effects (font (size 1.524 1.524)) hide)
+    )
+    (property "SolderPoints" "2" (id 5) (at 518.16 241.046 90)
+      (effects (font (size 1.524 1.524)) hide)
+    )
+  )
   (symbol (lib_id "Tittar_kl:L") (at 523.24 259.08 90) (unit 1)
     (in_bom yes) (on_board yes)
@@
     )
   )
+  (symbol (lib_id "Tittar_kl:C") (at 523.24 233.68 270) (unit 1)
+    (in_bom yes) (on_board yes)
+    (property "Reference" "C?" (id 0) (at 524.51 232.41 90)
+      (effects (font (size 1.27 1.27)) (justify left))
+    )
+    (property "Value" "2.2pF" (id 1) (at 520.7 229.87 90)
+      (effects (font (size 1.27 1.27)) (justify left))
+    )
+    (property "Footprint" "Capacitors:CAP_0402" (id 2) (at 519.43 236.22 90)
+      (effects (font (size 0.7112 0.7112)) (justify bottom) hide)
+    )
+    (property "Datasheet" "" (id 3) (at 523.24 233.68 0)
+      (effects (font (size 1.524 1.524)) hide)
+    )
+  )
   (symbol (lib_id "Tittar_kl:C") (at 530.86 265.43 0) (unit 1)
     (in_bom yes) (on_board yes)
@@
       (reference "#PWR0149") (unit 1) (value "PwrUnst") (footprint "")
     )
+    (path "/5ebd0a8b-3140-414d-a276-a357b7bf28e0"
+      (reference "#PWR?") (unit 1) (value "GND") (footprint "")
+    )
     (path "/5ddea526-9380-4d35-8754-24b2be7b263e"
       (reference "ANT1") (unit 1) (value "ANT_GENERAL") (footprint "Antennas:ANT_IFA_MUSHROOM")
@@
       (reference "C72") (unit 1) (value "10u") (footprint "Capacitors:CAP_0603_Silks")
     )
+    (path "/eca23a8e-6f78-4add-8598-ce57044d2ff7"
+      (reference "C?") (unit 1) (value "2.2pF") (footprint "Capacitors:CAP_0402")
+    )
     (path "/00000000-0000-0000-0000-000058014498"
       (reference "D1") (unit 1) (value "PMEG2020") (footprint "Diodes:SOD323")
@@
       (reference "L9") (unit 1) (value "BLM15AG102") (footprint "Inductors:IND_0402")
     )
+    (path "/e3345711-efbd-4159-99f8-da5257299204"
+      (reference "L?") (unit 1) (value "4.7nH") (footprint "Inductors:IND_0402")
+    )
     (path "/00000000-0000-0000-0000-00005937b7f9"
